File: pcb/pcehd.sch (KiCad schematic (older format))
At the start: 3 parts, among them U1 AP7361

Commit message: Expansion connection re-order for layout
Changed lines of the file:
@@
 F16 "RST_N" O R 7350 2150 60
 F17 "SPBG" I L 5850 2650 60
-F18 "D[0..7]" B L 5850 2050 60
-F19 "A[0..20]" I L 5850 2300 60
-F20 "VD[0..7]" I L 5850 2550 60
-F21 "R[4..0]" O R 7350 2500 60
-F22 "G[4..0]" O R 7350 2600 60
-F23 "B[4..0]" O R 7350 2700 60
-F24 "DCKFB" O L 5850 4200 60
-F25 "SI_CLK0" I L 5850 4300 60
-F26 "SI_CLK1" I L 5850 4400 60
+F18 "VD[0..7]" I L 5850 2550 60
+F19 "R[4..0]" O R 7350 2500 60
+F20 "G[4..0]" O R 7350 2600 60
+F21 "B[4..0]" O R 7350 2700 60
+F22 "DCKFB" O L 5850 4200 60
+F23 "SI_CLK0" I L 5850 4300 60
+F24 "SI_CLK1" I L 5850 4400 60
+F25 "D[7..0]" B L 5850 2050 60
+F26 "A[20..0]" I L 5850 2300 60
 $EndSheet
 $Sheet
@@
 F6 "CDD_I" I L 1600 2050 60
 F7 "CEK_O" O R 3100 3250 60
-F8 "D[0..7]" B R 3100 2050 60
-F9 "WR_N_O" O R 3100 3150 60
-F10 "A[0..20]" O R 3100 2300 60
-F11 "VD[0..7]" O R 3100 2550 60
-F12 "5V" I L 1600 4500 60
-F13 "DCK_O" O R 3100 3850 60
-F14 "HSn_O" O R 3100 4300 60
-F15 "CS_O" O R 3100 3350 60
+F8 "WR_N_O" O R 3100 3150 60
+F9 "VD[0..7]" O R 3100 2550 60
+F10 "5V" I L 1600 4500 60
+F11 "DCK_O" O R 3100 3850 60
+F12 "HSn_O" O R 3100 4300 60
+F13 "CS_O" O R 3100 3350 60
+F14 "D[7..0]" B R 3100 2050 60
+F15 "A[20..0]" O R 3100 2300 60
 $EndSheet
 Wire Wire Line

Commit message: New layout
Changed lines of the file:
@@
 Sheet 1 5
 Title "PCEHD"
-Date "2020-01-12"
+Date "2020-01-15"
 Rev "0.1"
 Comp ""
@@
 F13 "CEK" I L 5850 3250 60
 F14 "DDIR" O L 5850 2150 60
-F15 "CDD" O R 7350 2050 60
-F16 "RST_N" O R 7350 2150 60
-F17 "SPBG" I L 5850 2650 60
-F18 "VD[0..7]" I L 5850 2550 60
-F19 "R[4..0]" O R 7350 2500 60
-F20 "G[4..0]" O R 7350 2600 60
-F21 "B[4..0]" O R 7350 2700 60
-F22 "DCKFB" O L 5850 4200 60
-F23 "SI_CLK0" I L 5850 4300 60
-F24 "SI_CLK1" I L 5850 4400 60
-F25 "D[7..0]" B L 5850 2050 60
-F26 "A[20..0]" I L 5850 2300 60
+F15 "SPBG" I L 5850 2650 60
+F16 "VD[0..7]" I L 5850 2550 60
+F17 "DCKFB" O L 5850 4200 60
+F18 "SI_CLK0" I L 5850 4300 60
+F19 "SI_CLK1" I L 5850 4400 60
+F20 "D[7..0]" B L 5850 2050 60
+F21 "A[20..0]" I L 5850 2300 60
+F22 "XRD" I L 5850 3050 60
+F23 "HuID_N" I L 5850 2750 60
+F24 "HuID_N_O" O R 7350 2250 60
+F25 "RST_N_O" O R 7350 2150 60
+F26 "R[2..0]" O R 7350 2500 60
+F27 "G[2..0]" O R 7350 2600 60
+F28 "B[2..0]" O R 7350 2700 60
 $EndSheet
 $Sheet
@@
 F9 "DVDD3V3" I L 8600 5700 60
 F10 "5V" I L 8600 5600 60
-F11 "R[4..0]" I L 8600 2500 60
-F12 "G[4..0]" I L 8600 2600 60
-F13 "B[4..0]" I L 8600 2700 60
-F14 "I2S_DATA" I L 8600 5150 60
-F15 "I2S_BCK" I L 8600 5250 60
-F16 "I2S_WS" I L 8600 5350 60
+F11 "I2S_DATA" I L 8600 5150 60
+F12 "I2S_BCK" I L 8600 5250 60
+F13 "I2S_WS" I L 8600 5350 60
+F14 "R[2..0]" I L 8600 2500 60
+F15 "G[2..0]" I L 8600 2600 60
+F16 "B[2..0]" I L 8600 2700 60
 $EndSheet
 $Sheet
@@
 F4 "SPBG_O" O R 3100 2650 60
 F5 "DDIR_I" I R 3100 2150 60
-F6 "CDD_I" I L 1600 2050 60
-F7 "CEK_O" O R 3100 3250 60
-F8 "WR_N_O" O R 3100 3150 60
-F9 "VD[0..7]" O R 3100 2550 60
-F10 "5V" I L 1600 4500 60
-F11 "DCK_O" O R 3100 3850 60
-F12 "HSn_O" O R 3100 4300 60
-F13 "CS_O" O R 3100 3350 60
-F14 "D[7..0]" B R 3100 2050 60
-F15 "A[20..0]" O R 3100 2300 60
+F6 "CEK_O" O R 3100 3250 60
+F7 "WR_N_O" O R 3100 3150 60
+F8 "VD[0..7]" O R 3100 2550 60
+F9 "5V" I L 1600 4500 60
+F10 "DCK_O" O R 3100 3850 60
+F11 "HSn_O" O R 3100 4300 60
+F12 "CS_O" O R 3100 3350 60
+F13 "D[7..0]" B R 3100 2050 60
+F14 "A[20..0]" O R 3100 2300 60
+F15 "HuID_N_I" I L 1600 2250 60
+F16 "HuID_N_O" O R 3100 2750 60
+F17 "XRD_O" O R 3100 3050 60
 $EndSheet
 Wire Wire Line
@@
 Wire Wire Line
 	5200 5350 8600 5350
-Wire Wire Line
-	1600 2050 1400 2050
-Wire Wire Line
-	1400 2050 1400 1500
-Wire Wire Line
-	1400 1500 7650 1500
-Wire Wire Line
-	7650 1500 7650 2050
-Wire Wire Line
-	7650 2050 7350 2050
 Wire Wire Line
 	1600 2150 1350 2150
@@
 	7350 3600 8600 3600
 Wire Wire Line
-	5450 6100 6300 6100
+	5450 6100 5700 6100
+Wire Wire Line
+	7350 2250 7750 2250
+Wire Wire Line
+	7750 2250 7750 1400
+Wire Wire Line
+	7750 1400 1300 1400
+Wire Wire Line
+	1300 1400 1300 2250
+Wire Wire Line
+	1300 2250 1600 2250
+Wire Wire Line
+	3100 2750 5850 2750
+Wire Wire Line
+	3100 3050 5850 3050
+Wire Wire Line
+	5700 6050 5700 6100
+Connection ~ 5700 6100
+Wire Wire Line
+	5700 6100 6300 6100
 $EndSCHEMATC
