File: pcb/hdmitx.sch (KiCad schematic (older format))
At the start: 36 parts, among them J1 HDMI_CONN, U2 ADV7513, U3 TLV70018

Commit message: Finished initial schematic with audio
Parts:
- added C68, C78, C80, C81, C84, C85: 10u, custom_components:SM0603_Capa_libcms, symbol pcehd-rescue:C_Small-Device
- added C77, C79: 30p, custom_components:SM0603_Capa_libcms, symbol pcehd-rescue:C_Small-Device
- added C82, C83: 2.2u, custom_components:SM0603_Capa_libcms, symbol pcehd-rescue:C_Small-Device
- added R17, R19: 100k, custom_components:SM0603_Resistor_libcms, symbol ossc_board-rescue:R_Small
- added U14: PCM1862, custom_components:TSSOP-30_4.4x7.8mm_Pitch0.5mm_Handsoldering, symbol ossc_board-rescue:PCM1862
- added Y1: 24.576MHz, custom_components:ECS-3X9X, symbol ossc_board-rescue:Crystal_Small
Connections:
- wire segments 161 -> 191
- no-connect marks 3 -> 14
Other:
- moved on the sheet: D1, D2, D3, F1, J1, R3, R4, R5

Commit message: Cleaned up schematic, moved connections to busses
Connections:
- net labels added: B[4..0], G[4..0], R[4..0]
- net labels removed: B5, B6, B7, G5, G6, G7, R5, R6, R7
Other:
- moved on the sheet: R1, R2

Commit message: Added clock selection
Parts:
- removed C68, C78, C80, C81, C84, C85: 10u, custom_components:SM0603_Capa_libcms, symbol pcehd-rescue:C_Small-Device
- removed C77, C79: 30p, custom_components:SM0603_Capa_libcms, symbol pcehd-rescue:C_Small-Device
- removed C82, C83: 2.2u, custom_components:SM0603_Capa_libcms, symbol pcehd-rescue:C_Small-Device
- removed R17, R19: 100k, custom_components:SM0603_Resistor_libcms, symbol ossc_board-rescue:R_Small
- removed U14: PCM1862, custom_components:TSSOP-30_4.4x7.8mm_Pitch0.5mm_Handsoldering, symbol ossc_board-rescue:PCM1862
- removed Y1: 24.576MHz, custom_components:ECS-3X9X, symbol ossc_board-rescue:Crystal_Small
Connections:
- net labels removed: AudioL, AudioR
- wire segments 191 -> 161
- no-connect marks 14 -> 3
Other:
- moved on the sheet: D1, D2, D3, F1, J1, R1, R2, R3, R4, R5

Commit message: Added FS7140 PLL, moved to level-shift '245
Parts:
- U2: symbol HDMI:ADV7513 -> pcehd-rescue:ADV7513-HDMI
- U2: symbol HDMI:ADV7513 -> custom_components:ADV7513
Changed lines of the file:
@@
 $Descr A4 11693 8268
 encoding utf-8
-Sheet 5 5
+Sheet 3 5
 Title "PCEHD"
-Date "2020-01-03"
+Date "2020-01-12"
 Rev "0.1"
 Comp ""
@@
 5V
 $Comp
-L HDMI:ADV7513 U2
+L pcehd-rescue:ADV7513-HDMI U2
 U 1 1 5A38E9E6
 P 3750 6300
+AR Path="/5A38E9E6" Ref="U2"  Part="1"
+AR Path="/54FF6758/5A38E9E6" Ref="U2"  Part="1"
 F 0 "U2" H 3750 6450 50  0000 C CNN
 F 1 "ADV7513" H 3750 6350 50  0000 C CNN
@@
 $EndComp
 $Comp
-L HDMI:ADV7513 U2
+L custom_components:ADV7513 U2
 U 2 1 5A38EC28
 P 3800 950
@@
 	2650 2000 2800 2000
 Wire Wire Line
-	2200 1800 2800 1800
-Wire Wire Line
 	2200 1700 2800 1700
 Wire Wire Line
@@
 Text HLabel 2250 4050 0    60   Input ~ 0
 B[4..0]
+Text HLabel 2200 1300 0    60   Input ~ 0
+I2S_DATA
+Text HLabel 2200 1700 0    60   Input ~ 0
+I2S_BCK
+Text HLabel 2150 1800 0    60   Input ~ 0
+I2S_WS
+Wire Wire Line
+	2150 1800 2800 1800
 Wire Bus Line
 	2350 2350 2350 3050

Commit message: New layout
Connections:
- net labels added: B[2..0], G[2..0], R[2..0]
- net labels removed: B3, B4, B[4..0], G3, G4, G[4..0], R3, R4, R[4..0]
Changed lines of the file:
@@
 	2350 2350 2250 2350
 Text Label 2600 2450 0    60   ~ 0
-R4
+R2
 Text Label 2600 2550 0    60   ~ 0
-R3
+R1
 Text Label 2600 2650 0    60   ~ 0
+R0
+Text Label 2600 2750 0    60   ~ 0
 R2
-Text Label 2600 2750 0    60   ~ 0
+Text Label 2600 2850 0    60   ~ 0
 R1
-Text Label 2600 2850 0    60   ~ 0
+Text Label 2600 2950 0    60   ~ 0
 R0
-Text Label 2600 2950 0    60   ~ 0
-R4
 Text Label 2600 3050 0    60   ~ 0
-R3
+R2
 Text Label 2600 3150 0    60   ~ 0
-R2
+R1
 Text HLabel 2250 2350 0    60   Input ~ 0
-R[4..0]
+R[2..0]
 Entry Wire Line
 	2350 3900 2450 4000
@@
 	2450 4000 2800 4000
 Text Label 2600 3300 0    60   ~ 0
-G4
+G2
 Text Label 2600 3400 0    60   ~ 0
-G3
+G1
 Text Label 2600 3500 0    60   ~ 0
+G0
+Text Label 2600 3600 0    60   ~ 0
 G2
-Text Label 2600 3600 0    60   ~ 0
+Text Label 2600 3700 0    60   ~ 0
 G1
-Text Label 2600 3700 0    60   ~ 0
+Text Label 2600 3800 0    60   ~ 0
 G0
-Text Label 2600 3800 0    60   ~ 0
-G4
 Text Label 2600 3900 0    60   ~ 0
-G3
+G2
 Text Label 2600 4000 0    60   ~ 0
-G2
+G1
 Wire Bus Line
 	2350 3200 2250 3200
 Text HLabel 2250 3200 0    60   Input ~ 0
-G[4..0]
+G[2..0]
 Wire Wire Line
 	1900 5200 2800 5200
@@
 	2450 4850 2800 4850
 Text Label 2600 4150 0    60   ~ 0
-B4
+B2
 Text Label 2600 4250 0    60   ~ 0
-B3
+B1
 Text Label 2600 4350 0    60   ~ 0
+B0
+Text Label 2600 4450 0    60   ~ 0
 B2
-Text Label 2600 4450 0    60   ~ 0
+Text Label 2600 4550 0    60   ~ 0
 B1
-Text Label 2600 4550 0    60   ~ 0
+Text Label 2600 4650 0    60   ~ 0
 B0
-Text Label 2600 4650 0    60   ~ 0
-B4
 Text Label 2600 4750 0    60   ~ 0
-B3
+B2
 Text Label 2600 4850 0    60   ~ 0
-B2
+B1
 Wire Bus Line
 	2350 4050 2250 4050
 Text HLabel 2250 4050 0    60   Input ~ 0
-B[4..0]
+B[2..0]
 Text HLabel 2200 1300 0    60   Input ~ 0
 I2S_DATA
