File: pcb/pcehd.kicad_pcb (KiCad board)
At the start: 2 copper layers, 158 parts, among them J1 HDMI_CONN, P1 JTAG_CONN, Q1 BC847, Q2 BC847, U1 AP7361, U10 SN74LVCC4245APW, U11 SN74LVCC4245APW, U12 10CL025YE144C8N, U13 IS25LP016D-JBLE, U14 SN74LVCC4245APW, U15 TLV70012, U16 TLV70025, U17 TLV70012, U18 SN74LVCC4245APW, U19 SN74LVC3G17, U2 ADV7513, U3 TLV70018, U4 PCEngineExpansion, U5 FS7140-01G-XTD, U6 PCM1808PWR, U7 SI5351C-B, U8 74153, U9 SN74LVCC4245APW, Y1 25.000MHz

Commit message: Layout checkpoint
Parts:
- moved C84 109.8 mm to (126.5, 80.5)
- moved C85 103.1 mm to (117.1, 80.5)
- moved C89 101.8 mm to (135.4, 80.5)
- moved C81 95.6 mm to (126.2, 68.8)
- moved C88 94.4 mm to (135.4, 68.9)
- moved C23 88.1 mm to (103.9, 80.5)
- moved C90 82.4 mm to (105.4, 70.1), turned to 90 degrees
- moved C87 81.5 mm to (103.6, 68.8)
- moved C82 75.9 mm to (117.1, 68.8)
- moved Y1 73.5 mm to (105.2, 87.1), turned to 90 degrees
- moved C83 55.8 mm to (94.5, 68.8)
- moved C86 51.4 mm to (94.5, 80.5)
- moved U8 11.1 mm to (101.9, 108.0)
- moved U5 7.36 mm to (104.6, 96.3), turned to 0 degrees
- moved U12 6.90 mm to (106.7, 132.8)
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Routing:
- net /fpga1/D5: track 0.00 -> 77.9 mm, vias 0 -> 4
- net /fpga1/D7: track 0.00 -> 77.9 mm, vias 0 -> 4
- net /fpga1/D6: track 0.00 -> 77.5 mm, vias 0 -> 4
- net /fpga1/VD0: track 0.00 -> 71.6 mm
- net /fpga1/VD1: track 0.00 -> 70.3 mm
- net Net-(U19-Pad1): track 0.00 -> 69.8 mm, vias 0 -> 2
- net /fpga1/VD2: track 0.00 -> 69.3 mm
- net /fpga1/VD3: track 0.00 -> 68.4 mm
- net /fpga1/CEK: track 0.00 -> 68.0 mm
- net /fpga1/VD4: track 0.00 -> 67.6 mm
- net /fpga1/SPBG: track 0.00 -> 67.3 mm
- net /fpga1/VD5: track 0.00 -> 66.7 mm
- net /fpga1/A16: track 0.00 -> 66.7 mm
- net /fpga1/WR_N: track 0.00 -> 66.6 mm
- net /fpga1/VD6: track 0.00 -> 65.9 mm
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
Commit message: Layout check-in
Parts:
- moved P1 137.1 mm to (86.0, 162.4), turned to 180 degrees
- moved Q2 80.9 mm to (94.7, 99.6), turned to 90 degrees
- moved R22 78.6 mm to (96.9, 94.0)
- moved R24 77.1 mm to (95.4, 103.8)
- moved R25 70.1 mm to (93.7, 103.8)
- moved R23 68.0 mm to (95.2, 94.0)
- moved R18 61.6 mm to (85.1, 111.3), turned to 180 degrees
- moved Q1 59.5 mm to (96.3, 89.7), turned to 90 degrees
- moved R28 55.8 mm to (65.7, 106.8)
- moved R15 54.8 mm to (87.6, 129.0), turned to 180 degrees
- moved R16 53.0 mm to (87.1, 125.2)
- moved C73 48.2 mm to (83.3, 113.0), turned to 0 degrees
- moved U13 34.4 mm to (86.1, 118.4), turned to 90 degrees
- moved J1 14.4 mm to (106.7, 177.3), turned to 0 degrees
- moved U2 7.77 mm to (106.7, 158.8)
Routing:
- net /hdmitx1/I2S_WS: track 0.00 -> 97.3 mm, vias 0 -> 2
- net /hdmitx1/I2S_BCK: track 0.00 -> 90.5 mm, vias 0 -> 2
- net Net-(Q2-Pad3): track 0.00 -> 88.8 mm, vias 0 -> 4
- net /hdmitx1/I2S_DATA: track 0.00 -> 88.2 mm, vias 0 -> 2
- net /fpga1/CDD: track 0.00 -> 48.7 mm, vias 0 -> 2
- net Net-(Q1-Pad3): track 0.00 -> 45.4 mm, vias 0 -> 2
- net /fpga1/RST_N: track 0.00 -> 40.2 mm, vias 0 -> 2
- net /fpga1/TCK: track 0.00 -> 38.6 mm, vias 0 -> 1
- net /fpga1/TDO: track 0.00 -> 34.1 mm, vias 0 -> 1
- net /fpga1/TMS: track 0.00 -> 33.0 mm, vias 0 -> 1
- net /fpga1/DCKFB: track 0.00 -> 32.1 mm, vias 0 -> 2
- net /fpga1/TDI: track 0.00 -> 30.3 mm, vias 0 -> 1
- net (no net): track 0.00 -> 29.6 mm, vias 0 -> 1
- net /fpga1/R1: track 0.00 -> 27.1 mm
- net /fpga1/R0: track 0.00 -> 25.3 mm
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
Commit message: New layout
Parts:
- added C91: 0.1u, custom_components:SM0603_Capa_libcms, F.Cu at (159.3, 49.8)
- added C92: 0.1u, custom_components:SM0603_Capa_libcms, F.Cu at (158.2, 61.7)
- added J2: Micro_SD_Card, Connector_Card:microSD_HC_Hirose_DM3D-SF, F.Cu at (97.2, 99.8)
- added R30: 10K, custom_components:SM0603_Resistor_libcms, F.Cu at (204.6, 33.7)
- added U20: SN74LVC2G17, custom_components:SOT-23-6_Handsoldering, F.Cu at (130.6, 56.1)
- R22: value 1K -> 10K
- R23: value 10K -> 1K
- U19: value SN74LVC3G17 -> SN74LVCC4245APW; footprint custom_components:SSOP-8_3x3mm_Pitch0.65mm -> custom_components:SN74LVCC4245APW
- moved R21 234.8 mm to (-40.1, 75.9), turned to 0 degrees
- moved C2 205.8 mm to (221.8, 26.6), turned to 0 degrees
- moved C25 204.0 mm to (-40.1, 81.1), turned to 0 degrees
- moved C1 203.8 mm to (221.8, 29.2), turned to 0 degrees
- moved R20 202.2 mm to (-43.7, 78.2), turned to 0 degrees
- moved U1 195.9 mm to (216.1, 30.6), turned to 0 degrees
- moved C68 195.9 mm to (-43.7, 81.0), turned to 0 degrees
- moved C79 193.8 mm to (-32.9, 75.8), turned to 0 degrees
- moved JP6 193.1 mm to (-21.7, 75.2), turned to 0 degrees
- moved R6 191.7 mm to (-40.1, 78.5), turned to 0 degrees
- moved JP4 191.1 mm to (-26.1, 74.7), turned to 0 degrees
- moved C24 187.1 mm to (-36.5, 78.5), turned to 0 degrees
- moved JP5 186.6 mm to (-21.7, 71.6), turned to 0 degrees
- moved C80 185.7 mm to (-36.5, 75.9), turned to 0 degrees
- moved D4 184.3 mm to (-3.52, 64.6), turned to 0 degrees
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Connections:
- net /fpga1/RST_N renamed /input1/RST_N_I
- net Net-(Q2-Pad3) renamed /input1/RSTn
- net Net-(U11-Pad8) renamed /input1/WRn
- Q1 pad 3: Net-(Q1-Pad3) -> /input1/HuID
- R22 pad 1: Net-(Q1-Pad1) -> /5V
- R22 pad 2: /fpga1/CDD -> Net-(R22-Pad2)
- R23 pad 2: GND -> /input1/HuID_N_I
- U10 pad 14: /fpga1/A8 -> /fpga1/A18
- U10 pad 15: /fpga1/A13 -> /fpga1/A14
- U10 pad 16: /fpga1/A10 -> /fpga1/A17
- U10 pad 17: /fpga1/A11 -> /fpga1/A9
- U10 pad 18: /fpga1/A0 -> /fpga1/A8
- U10 pad 19: /fpga1/A2 -> /fpga1/A13
- U10 pad 20: /fpga1/A1 -> /fpga1/A10
- U10 pad 21: /fpga1/A3 -> /fpga1/A11
- U11 pad 10: /input1/CEK -> /input1/CS
- U11 pad 14: /fpga1/CEK -> /fpga1/CS
- U11 pad 15: /fpga1/SPBG -> /fpga1/HuID_N
- U11 pad 17: /fpga1/A20 -> /fpga1/CEK
- U11 pad 18: /fpga1/A18 -> (no net)
- U11 pad 19: /fpga1/A14 -> /fpga1/XRD
- U11 pad 20: /fpga1/A17 -> (no net)
- U11 pad 21: /fpga1/A9 -> (no net)
- U11 pad 3: Net-(U11-Pad3) -> (no net)
- U11 pad 4: Net-(U11-Pad4) -> /input1/VSn
- U11 pad 5: Net-(U11-Pad5) -> /input1/XRD
- U11 pad 6: Net-(U11-Pad6) -> /input1/XNMI
- U11 pad 7: Net-(U11-Pad7) -> /input1/CEK
- U11 pad 9: /input1/SPBG -> /input1/HuID
- U12 pad 22: (no net) -> /fpga1/XRD
- U12 pad 28: /fpga1/CDD -> /input1/HuID_N_I
- U12 pad 32: /fpga1/SDA -> /fpga1/DAT1
- U12 pad 33: /fpga1/SCL -> /fpga1/DAT0
- U12 pad 39: /fpga1/HDMITX_VSYNC -> /fpga1/SCLK
- U12 pad 42: /fpga1/HDMITX_HSYNC -> /fpga1/CMD
- U12 pad 43: /hdmitx1/DE -> /fpga1/DAT3
- U12 pad 44: /fpga1/B2 -> /fpga1/DAT2
- U12 pad 46: /fpga1/B3 -> /fpga1/HDMITX_VSYNC
- U12 pad 49: /fpga1/B4 -> /fpga1/HDMITX_HSYNC
- U12 pad 50: /fpga1/B0 -> /hdmitx1/DE
- U12 pad 51: /fpga1/B1 -> /fpga1/B2
- U12 pad 54: (no net) -> /fpga1/HuID_N
- U12 pad 58: /fpga1/G2 -> /fpga1/B0
- U12 pad 60: /fpga1/G3 -> /fpga1/B1
- U12 pad 66: /fpga1/G4 -> /fpga1/G2
- U12 pad 71: /fpga1/R3 -> /fpga1/R0
- U12 pad 72: /fpga1/R4 -> /fpga1/R1
- U12 pad 76: /fpga1/R0 -> /fpga1/SCL
- U12 pad 77: /fpga1/R1 -> /fpga1/SDA
- U19 pad 1: Net-(U19-Pad1) -> /5V
- U19 pad 2: /input2/HSn -> Net-(R22-Pad2)
- U19 pad 4: GND -> /input1/RDYn
- U19 pad 5: /fpga1/DCK -> Net-(U19-Pad5)
- U19 pad 6: /input1/HSn -> Net-(U19-Pad6)
- U19 pad 7: /fpga1/CS -> Net-(U19-Pad7)
- U19 pad 8: VCC -> Net-(U19-Pad8)
- U2 pad 37: /fpga1/R4 -> /fpga1/R2
- U2 pad 38: /fpga1/R3 -> /fpga1/R1
- U2 pad 39: /fpga1/R2 -> /fpga1/R0
- U2 pad 40: /fpga1/R1 -> /fpga1/R2
- U2 pad 41: /fpga1/R0 -> /fpga1/R1
- U2 pad 42: /fpga1/R4 -> /fpga1/R0
- U2 pad 43: /fpga1/R3 -> /fpga1/R2
- U2 pad 44: /fpga1/R2 -> /fpga1/R1
- U2 pad 45: /fpga1/G4 -> /fpga1/G2
- U2 pad 46: /fpga1/G3 -> /fpga1/G1
- U2 pad 47: /fpga1/G2 -> /fpga1/G0
- U2 pad 48: /fpga1/G1 -> /fpga1/G2
- U2 pad 49: /fpga1/G0 -> /fpga1/G1
- U2 pad 50: /fpga1/G4 -> /fpga1/G0
- U2 pad 52: /fpga1/G3 -> /fpga1/G2
- U2 pad 54: /fpga1/G2 -> /fpga1/G1
- U2 pad 55: /fpga1/B4 -> /fpga1/B2
- U2 pad 56: /fpga1/B3 -> /fpga1/B1
- U2 pad 57: /fpga1/B2 -> /fpga1/B0
- U2 pad 58: /fpga1/B1 -> /fpga1/B2
- U2 pad 59: /fpga1/B0 -> /fpga1/B1
- U2 pad 60: /fpga1/B4 -> /fpga1/B0
- U2 pad 61: /fpga1/B3 -> /fpga1/B2
- U2 pad 62: /fpga1/B2 -> /fpga1/B1
- U4 pad A10: (no net) -> /input1/VSn
- U4 pad A3: Net-(U19-Pad1) -> /input1/CS
- U4 pad A4: Net-(U11-Pad6) -> Net-(U10-Pad10)
- U4 pad A5: Net-(U11-Pad5) -> Net-(U10-Pad9)
- U4 pad A6: Net-(U11-Pad3) -> Net-(U10-Pad7)
- U4 pad A7: Net-(U10-Pad8) -> Net-(U10-Pad4)
- U4 pad A9: Net-(U19-Pad3) -> /input1/DCK
- U4 pad B12: Net-(U10-Pad6) -> Net-(U4-PadB12)
- U4 pad B13: Net-(U10-Pad5) -> Net-(U4-PadB13)
- U4 pad B17: Net-(U4-PadB17) -> Net-(U19-Pad9)
- U4 pad B18: Net-(U4-PadB18) -> Net-(U19-Pad8)
- U4 pad B19: Net-(U11-Pad7) -> Net-(U19-Pad5)
- U4 pad B2: Net-(Q1-Pad3) -> (no net)
- U4 pad B20: (no net) -> /input1/RDYn
- U4 pad B21: (no net) -> Net-(U19-Pad3)
- U4 pad B5: (no net) -> /input1/XNMI
- U4 pad B6: Net-(U10-Pad10) -> Net-(U10-Pad6)
- U4 pad B7: (no net) -> /input1/XRD
- U4 pad C13: Net-(U10-Pad4) -> Net-(U4-PadC13)
- U4 pad C14: Net-(U10-Pad3) -> Net-(U4-PadC14)
- U4 pad C16: Net-(U4-PadC16) -> Net-(U19-Pad10)
- U4 pad C18: Net-(U4-PadC18) -> Net-(U19-Pad7)
- U4 pad C19: Net-(U4-PadC19) -> Net-(U19-Pad6)
- U4 pad C3: (no net) -> /input1/HuID
- U4 pad C5: Net-(U11-Pad4) -> Net-(U10-Pad8)
- U4 pad C6: Net-(U10-Pad9) -> Net-(U10-Pad5)
- U4 pad C7: Net-(U10-Pad7) -> Net-(U10-Pad3)
- U9 pad 10: Net-(U4-PadB15) -> /input1/SPBG
- U9 pad 14: /fpga1/A5 -> /fpga1/SPBG
- U9 pad 15: /fpga1/A4 -> /fpga1/A0
- U9 pad 16: /fpga1/A7 -> /fpga1/A2
- U9 pad 17: /fpga1/A6 -> /fpga1/A1
- U9 pad 18: /fpga1/A12 -> /fpga1/A3
- U9 pad 19: /fpga1/A16 -> /fpga1/A5
- U9 pad 20: /fpga1/A15 -> /fpga1/A4
- U9 pad 21: /fpga1/A19 -> /fpga1/A7
- U9 pad 3: Net-(U4-PadC19) -> Net-(U4-PadB16)
- U9 pad 4: Net-(U4-PadC18) -> Net-(U4-PadC15)
- U9 pad 5: Net-(U4-PadB18) -> Net-(U4-PadB15)
- U9 pad 6: Net-(U4-PadB17) -> Net-(U4-PadC14)
- U9 pad 7: Net-(U4-PadC16) -> Net-(U4-PadC13)
- U9 pad 8: Net-(U4-PadB16) -> Net-(U4-PadB13)
- U9 pad 9: Net-(U4-PadC15) -> Net-(U4-PadB12)
Routing:
- net /hdmitx1/I2S_WS: track 97.3 -> 0.00 mm, vias 2 -> 0
- net /hdmitx1/I2S_BCK: track 90.5 -> 0.00 mm, vias 2 -> 0
- net /input1/RSTn: track 88.8 -> 0.00 mm, vias 4 -> 0
- net /hdmitx1/I2S_DATA: track 88.2 -> 0.00 mm, vias 2 -> 0
- net /fpga1/D5: track 77.9 -> 0.00 mm, vias 4 -> 0
- net /fpga1/D7: track 77.9 -> 0.00 mm, vias 4 -> 0
- net /fpga1/D6: track 77.5 -> 0.00 mm, vias 4 -> 0
- net /fpga1/CEK: track 75.1 -> 0.00 mm
- net /fpga1/SPBG: track 74.5 -> 0.00 mm
- net /fpga1/WR_N: track 73.8 -> 0.00 mm
- net /fpga1/VD0: track 71.6 -> 0.00 mm
- net /fpga1/VD1: track 70.3 -> 0.00 mm
- net Net-(U19-Pad1): track 69.8 -> 0.00 mm, vias 2 -> 0
- net /fpga1/VD2: track 69.3 -> 0.00 mm
- net /fpga1/VD3: track 68.4 -> 0.00 mm
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Other:
- board outline added: 118.2 x 73.2 mm

Commit message: New layout checkpoint
Parts:
- moved U5 138.6 mm to (97.3, 74.4), turned to 180 degrees
- moved U8 130.8 mm to (97.3, 85.6)
- moved D2 120.2 mm to (166.6, 92.4), turned to 180 degrees
- moved D3 110.2 mm to (163.7, 92.5), turned to 180 degrees
- moved U7 106.5 mm to (97.3, 65.5)
- moved C29 81.8 mm to (32.4, 131.5)
- moved C68 81.8 mm to (18.0, 134.7)
- moved C77 81.8 mm to (32.4, 134.0)
- moved JP3 81.8 mm to (49.2, 124.8)
- moved R20 81.8 mm to (18.0, 132.0)
- moved U6 81.8 mm to (38.0, 120.2)
- moved Y1 81.8 mm to (46.0, 119.6)
- moved C24 81.8 mm to (25.2, 132.3)
- moved C26 81.8 mm to (25.2, 134.8)
- moved C27 81.8 mm to (28.8, 134.7)
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Connections:
- J1 pad 13: (no net) -> Net-(J1-Pad13)
- J1 pad 14: (no net) -> Net-(J1-Pad14)
- P1 pad 6: (no net) -> Net-(P1-Pad6)
- P1 pad 7: (no net) -> Net-(P1-Pad7)
- P1 pad 8: (no net) -> Net-(P1-Pad8)
- U10 pad 23: (no net) -> Net-(U10-Pad23)
- U11 pad 18: (no net) -> Net-(U11-Pad18)
- U11 pad 20: (no net) -> Net-(U11-Pad20)
- U11 pad 21: (no net) -> Net-(U11-Pad21)
- U11 pad 23: (no net) -> Net-(U11-Pad23)
- U11 pad 3: (no net) -> Net-(U11-Pad3)
- U12 pad 10: /fpga1/DDIR -> /fpga1/A10
- U12 pad 100: /fpga1/A7 -> /fpga1/VD3
- U12 pad 101: /fpga1/A4 -> /fpga1/VD4
- U12 pad 103: /fpga1/A5 -> /fpga1/VD5
- U12 pad 105: /fpga1/A3 -> /fpga1/VD6
- U12 pad 106: /fpga1/A1 -> /fpga1/VD7
- U12 pad 11: /fpga1/DCKFB -> /fpga1/A13
- U12 pad 111: /fpga1/A2 -> /fpga1/SCL
- U12 pad 112: /fpga1/A0 -> /fpga1/SDA
- U12 pad 113: /fpga1/A11 -> /fpga1/A7
- U12 pad 114: /fpga1/A10 -> /fpga1/A4
- U12 pad 115: /fpga1/A13 -> /fpga1/A5
- U12 pad 119: /fpga1/A8 -> /fpga1/A3
- U12 pad 120: /fpga1/D7 -> /fpga1/A1
- U12 pad 121: /fpga1/D6 -> /fpga1/A2
- U12 pad 125: /fpga1/D5 -> /fpga1/A0
- U12 pad 128: /fpga1/DCK -> /fpga1/SPBG
- U12 pad 129: /fpga1/CS -> /fpga1/DCK
- U12 pad 132: /fpga1/D4 -> /input1/HuID_N_I
- U12 pad 133: /fpga1/D3 -> /fpga1/D7
- U12 pad 135: /fpga1/D2 -> /fpga1/D6
- U12 pad 136: /fpga1/D1 -> /fpga1/D5
- U12 pad 137: /fpga1/D0 -> /fpga1/D4
- U12 pad 141: /fpga1/A9 -> /fpga1/D3
- U12 pad 142: /fpga1/A17 -> /fpga1/D2
- U12 pad 143: /fpga1/A14 -> /fpga1/D1
- U12 pad 144: /fpga1/A18 -> /fpga1/D0
- U12 pad 22: /fpga1/XRD -> /fpga1/A8
- U12 pad 23: /fpga1/WR_N -> /fpga1/A9
- U12 pad 24: /fpga1/SPBG -> /fpga1/A17
- U12 pad 25: /fpga1/CEK -> /fpga1/A14
- U12 pad 28: /input1/HuID_N_I -> /fpga1/A18
- U12 pad 31: /input1/RST_N_I -> /fpga1/XRD
- U12 pad 46: /fpga1/HDMITX_VSYNC -> Net-(U12-Pad46)
- U12 pad 49: /fpga1/HDMITX_HSYNC -> /input1/RST_N_I
- U12 pad 50: /hdmitx1/DE -> /fpga1/DCKFB
- U12 pad 51: /fpga1/B2 -> /fpga1/DDIR
- U12 pad 52: /fpga1/A19 -> /fpga1/CEK
- U12 pad 53: /fpga1/A15 -> /fpga1/WR_N
- U12 pad 55: (no net) -> /fpga1/CS
- U12 pad 58: /fpga1/B0 -> /fpga1/HDMITX_INT_N
- U12 pad 59: /fpga1/HDMITX_PCLK -> /fpga1/HDMITX_VSYNC
- U12 pad 60: /fpga1/B1 -> /fpga1/HDMITX_HSYNC
- U12 pad 65: /fpga1/HDMITX_INT_N -> /hdmitx1/DE
- U12 pad 66: /fpga1/G2 -> /fpga1/B0
- U12 pad 67: /fpga1/G0 -> /fpga1/B1
- U12 pad 68: /fpga1/G1 -> /fpga1/B2
- U12 pad 69: /fpga1/R2 -> /fpga1/HDMITX_PCLK
- U12 pad 7: /fpga1/A20 -> /fpga1/A11
- U12 pad 71: /fpga1/R0 -> /fpga1/G0
- U12 pad 72: /fpga1/R1 -> /fpga1/G1
- U12 pad 76: /fpga1/SCL -> /fpga1/G2
- U12 pad 77: /fpga1/SDA -> /fpga1/R0
- U12 pad 80: /fpga1/VD0 -> /fpga1/R1
- U12 pad 83: /fpga1/VD1 -> /fpga1/R2
- U12 pad 85: /fpga1/VD2 -> /fpga1/A20
- U12 pad 86: /fpga1/VD3 -> /fpga1/A19
- U12 pad 87: /fpga1/VD4 -> /fpga1/A15
- U12 pad 88: /fpga1/VD5 -> /fpga1/A16
- U12 pad 89: /fpga1/VD6 -> /fpga1/A12
- U12 pad 90: /fpga1/VD7 -> /fpga1/A6
- U12 pad 91: /fpga1/A16 -> /fpga1/VD0
- U12 pad 98: /fpga1/A12 -> /fpga1/VD1
- U12 pad 99: /fpga1/A6 -> /fpga1/VD2
- U14 pad 23: (no net) -> Net-(U14-Pad23)
- U15 pad 4: (no net) -> Net-(U15-Pad4)
- U16 pad 4: (no net) -> Net-(U16-Pad4)
- U17 pad 4: (no net) -> Net-(U17-Pad4)
- U18 pad 23: (no net) -> Net-(U18-Pad23)
- U19 pad 20: (no net) -> Net-(U19-Pad20)
- U19 pad 21: (no net) -> Net-(U19-Pad21)
- U19 pad 23: (no net) -> Net-(U19-Pad23)
- U2 pad 30: (no net) -> Net-(U2-Pad30)
- U3 pad 4: (no net) -> Net-(U3-Pad4)
- U4 pad A11: (no net) -> Net-(U4-PadA11)
- U4 pad A14: (no net) -> Net-(U4-PadA14)
- U4 pad A22: (no net) -> Net-(U4-PadA22)
- U4 pad A23: (no net) -> Net-(U4-PadA23)
- U4 pad B1: (no net) -> Net-(U4-PadB1)
- U4 pad B2: (no net) -> Net-(U4-PadB2)
- U4 pad B23: (no net) -> Net-(U4-PadB23)
- U4 pad B3: (no net) -> Net-(U4-PadB3)
- U4 pad C22: (no net) -> Net-(U4-PadC22)
- U4 pad C23: (no net) -> Net-(U4-PadC23)
- U5 pad 10: (no net) -> Net-(U5-Pad10)
- U5 pad 13: (no net) -> Net-(U5-Pad13)
- U5 pad 5: (no net) -> Net-(U5-Pad5)
- U5 pad 6: (no net) -> Net-(U5-Pad6)
- U5 pad 9: (no net) -> Net-(U5-Pad9)
- U7 pad 15: (no net) -> Net-(U7-Pad15)
- U7 pad 16: (no net) -> Net-(U7-Pad16)
- U7 pad 17: (no net) -> Net-(U7-Pad17)
- U7 pad 8: (no net) -> Net-(U7-Pad8)
- U7 pad 9: (no net) -> Net-(U7-Pad9)
- U8 pad 10: (no net) -> Net-(U8-Pad10)
- U8 pad 11: (no net) -> Net-(U8-Pad11)
- U8 pad 12: (no net) -> Net-(U8-Pad12)
- U8 pad 13: (no net) -> Net-(U8-Pad13)
- U8 pad 9: (no net) -> Net-(U8-Pad9)
- U9 pad 23: (no net) -> Net-(U9-Pad23)
Routing:
- net /fpga1/DCK: track 0.00 -> 74.5 mm, vias 0 -> 2
- net /fpga1/CS: track 0.00 -> 65.6 mm, vias 0 -> 2
- net /fpga1/WR_N: track 0.00 -> 65.3 mm, vias 0 -> 2
- net /fpga1/HuID_N: track 0.00 -> 65.2 mm, vias 0 -> 2
- net /fpga1/CEK: track 0.00 -> 65.2 mm, vias 0 -> 2
- net /fpga1/R2: track 0.00 -> 63.5 mm
- net /fpga1/R1: track 0.00 -> 61.2 mm
- net /fpga1/A18: track 0.00 -> 60.3 mm
- net /input2/HSn: track 0.00 -> 59.0 mm, vias 0 -> 2
- net /fpga1/XRD: track 0.00 -> 58.9 mm, vias 0 -> 2
- net /fpga1/R0: track 0.00 -> 58.9 mm
- net /fpga1/A14: track 0.00 -> 58.6 mm
- net /fpga1/A17: track 0.00 -> 57.5 mm
- net /fpga1/A9: track 0.00 -> 56.5 mm
- net /fpga1/G1: track 0.00 -> 56.4 mm
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Other:
- board size 118.2 x 73.2 mm -> 118.2 x 73 mm

Commit message: New layout checkpoint
Parts:
- moved U13 161.1 mm to (151.4, 92.6)
- moved C73 155.9 mm to (155.2, 87.8), turned to 270 degrees
- moved R16 155.8 mm to (145.4, 92.8), turned to 180 degrees
- moved R30 154.1 mm to (97.2, 50.6), turned to 270 degrees
- moved R10 153.7 mm to (170.0, 69.4), turned to 270 degrees
- moved R23 151.4 mm to (95.4, 50.6), turned to 270 degrees
- moved C78 150.0 mm to (101.6, 63.6), turned to 180 degrees
- moved R18 145.4 mm to (157.0, 87.8), turned to 270 degrees
- moved R9 140.5 mm to (172.0, 69.4), turned to 270 degrees
- moved D4 131.9 mm to (164.2, 39.8), turned to 270 degrees
- moved R12 127.1 mm to (87.6, 66.4), turned to 270 degrees
- moved R13 124.2 mm to (89.4, 66.4), turned to 270 degrees
- moved C90 123.2 mm to (129.8, 60.4), turned to 270 degrees
- moved C68 118.1 mm to (90.2, 41.2), turned to 180 degrees
- moved C25 118.0 mm to (96.8, 44.0), turned to 90 degrees
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Connections:
- J1 pad 13: Net-(J1-Pad13) -> (no net)
- J1 pad 14: Net-(J1-Pad14) -> (no net)
- P1 pad 6: Net-(P1-Pad6) -> (no net)
- P1 pad 7: Net-(P1-Pad7) -> (no net)
- P1 pad 8: Net-(P1-Pad8) -> (no net)
- U10 pad 23: Net-(U10-Pad23) -> (no net)
- U11 pad 18: Net-(U11-Pad18) -> (no net)
- U11 pad 20: Net-(U11-Pad20) -> (no net)
- U11 pad 21: Net-(U11-Pad21) -> (no net)
- U11 pad 23: Net-(U11-Pad23) -> (no net)
- U11 pad 3: Net-(U11-Pad3) -> (no net)
- U12 pad 46: Net-(U12-Pad46) -> (no net)
- U14 pad 23: Net-(U14-Pad23) -> (no net)
- U15 pad 4: Net-(U15-Pad4) -> (no net)
- U16 pad 4: Net-(U16-Pad4) -> (no net)
- U17 pad 4: Net-(U17-Pad4) -> (no net)
- U18 pad 23: Net-(U18-Pad23) -> (no net)
- U19 pad 20: Net-(U19-Pad20) -> (no net)
- U19 pad 21: Net-(U19-Pad21) -> (no net)
- U19 pad 23: Net-(U19-Pad23) -> (no net)
- U2 pad 30: Net-(U2-Pad30) -> (no net)
- U3 pad 4: Net-(U3-Pad4) -> (no net)
- U4 pad A11: Net-(U4-PadA11) -> (no net)
- U4 pad A14: Net-(U4-PadA14) -> (no net)
- U4 pad A22: Net-(U4-PadA22) -> (no net)
- U4 pad A23: Net-(U4-PadA23) -> (no net)
- U4 pad B1: Net-(U4-PadB1) -> (no net)
- U4 pad B2: Net-(U4-PadB2) -> (no net)
- U4 pad B23: Net-(U4-PadB23) -> (no net)
- U4 pad B3: Net-(U4-PadB3) -> (no net)
- U4 pad C22: Net-(U4-PadC22) -> (no net)
- U4 pad C23: Net-(U4-PadC23) -> (no net)
- U5 pad 10: Net-(U5-Pad10) -> (no net)
- U5 pad 13: Net-(U5-Pad13) -> (no net)
- U5 pad 5: Net-(U5-Pad5) -> (no net)
- U5 pad 6: Net-(U5-Pad6) -> (no net)
- U5 pad 9: Net-(U5-Pad9) -> (no net)
- U7 pad 15: Net-(U7-Pad15) -> (no net)
- U7 pad 16: Net-(U7-Pad16) -> (no net)
- U7 pad 17: Net-(U7-Pad17) -> (no net)
- U7 pad 8: Net-(U7-Pad8) -> (no net)
- U7 pad 9: Net-(U7-Pad9) -> (no net)
- U8 pad 10: Net-(U8-Pad10) -> (no net)
- U8 pad 11: Net-(U8-Pad11) -> (no net)
- U8 pad 12: Net-(U8-Pad12) -> (no net)
- U8 pad 13: Net-(U8-Pad13) -> (no net)
- U8 pad 9: Net-(U8-Pad9) -> (no net)
- U9 pad 23: Net-(U9-Pad23) -> (no net)
Routing:
- net VCC: track 0.00 -> 159.8 mm, vias 0 -> 4
- net /hdmitx1/I2S_WS: track 0.00 -> 148.1 mm, vias 0 -> 4
- net /5V: track 0.00 -> 147.0 mm, vias 0 -> 7
- net /hdmitx1/I2S_BCK: track 0.00 -> 136.7 mm, vias 0 -> 4
- net /hdmitx1/I2S_DATA: track 0.00 -> 132.6 mm, vias 0 -> 4
- net /fpga1/DDIR: track 0.00 -> 129.9 mm, vias 0 -> 4
- net /fpga1/SCL: track 0.00 -> 128.7 mm, vias 0 -> 4
- net /fpga1/SDA: track 0.00 -> 120.9 mm, vias 0 -> 4
- net /fpga1/TMS: track 0.00 -> 102.7 mm, vias 0 -> 2
- net /input1/RST_N_I: track 0.00 -> 97.0 mm, vias 0 -> 4
- net /fpga1/TDO: track 0.00 -> 89.3 mm, vias 0 -> 2
- net /fpga1/TCK: track 0.00 -> 74.2 mm, vias 0 -> 2
- net Net-(R26-Pad2): track 0.00 -> 68.6 mm
- net /fpga1/ASDO: track 0.00 -> 61.6 mm, vias 0 -> 2
- net /fpga1/TDI: track 0.00 -> 60.3 mm, vias 0 -> 2
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- added copper zone on B.Cu, net GNDREF
- added copper zone on F.Cu, net GNDREF
Other:
- net class Power added: clearance 0.2, trace_width 0.35, via_dia 1, via_drill 0.4
