File: pcb/input2.sch (KiCad schematic (older format))
At the start: 31 parts, among them U4 PCEngineExpansion, U5 FS7140-01G-XTD, U6 PCM1808PWR, U7 SI5351C-B, U8 74153, Y1 25.000MHz

Commit message: Finished version 0.1
Connections:
- net labels removed: HSn
Changed lines of the file:
@@
 DCK
 Text HLabel 1650 5700 0    60   Input ~ 0
-HSn
+HSn_buf
 Text Label 1950 5700 0    60   ~ 0
 HSn_buf
